Commit message: modified for ur5+franka simulation

File: franka_description/robots/panda_arm.xacro (robot description, xacro)
@@ -5,5 +5,6 @@
   <xacro:macro name="panda_arm" params="arm_id:='panda' description_pkg:='franka_description' connected_to:='' xyz:='0 0 0' rpy:='0 0 0' safety_distance:=0">
     <xacro:unless value="${not connected_to}">
-      <joint name="${arm_id}_joint_${connected_to}" type="fixed">
+      <!-- <joint name="${arm_id}_joint_${connected_to}" type="fixed"> -->
+      <joint name="${connected_to}_joint" type="fixed">
         <parent link="${connected_to}"/>
         <child link="${arm_id}_link0"/>
